Commit message: Added goal facet option

File: assets/urdf/objects/large_cube.urdf (robot description, URDF)
Before this commit: robot large_cube, 1 links, 0 joints
Links:
- removed link cube_body
- added link object, mass 0.723168; collision box size=0.09 0.09 0.09; visual mesh filename=meshes/large_cube.obj scale=1 1 1

File: assets/urdf/objects/small_cube.urdf (robot description, URDF)
Before this commit: robot small_cube, 1 links, 0 joints
Links:
- removed link cube_body
- added link small_cube, mass 0.035; collision mesh filename=meshes/small_cube.obj scale=1 1 1; visual mesh filename=meshes/small_cube.obj scale=1 1 1

File: assets/urdf/objects/small_cylinder.urdf (robot description, URDF)
Before this commit: robot small_cylinder, 1 links, 0 joints
Links:
- removed link cylinder_body
- added link object, mass 0.224385; collision cylinder length=0.08 radius=0.03; visual mesh filename=meshes/small_cylinder.obj scale=1 1 1
